File: RC-Bandpass-(.ac)/RC-Bandpass-(.ac).kicad_sch (KiCad schematic)
At the start: 5 parts

Commit message: Updated all schematics and prepared for KiCad 8.0
Parts:
- C1: value 10u -> 100u
- R1: value 10 -> 100
