File: Rectifier-4D-Regulator-(.tran)/Rectifier-4D-Regulator-(.tran).kicad_sch (KiCad schematic)
At the start: 13 parts, among them U1 LM317_TO-220

Commit message: Updated all schematics and prepared for KiCad 8.0
Parts:
- C1: value 3300u -> 4700u
- D1, D2, D3, D4: value 1N5408 -> D
- R2: value 360 -> 746
- Rload1: value 5 -> 8
Connections:
- net Vi renamed Vin
Other:
- note added: ".tran .1m 100m"
- note removed: ".tran .1m 200m"
