File: Rectifier-4D-Regulator-PNP-(.tran)/Rectifier-4D-Regulator-PNP-(.tran).kicad_sch (KiCad schematic)
At the start: 15 parts, among them Q1 BDX54C, U1 LM317_TO-220

Commit message: Updated all schematics and prepared for KiCad 8.0
Parts:
- removed Q1: BDX54C, symbol Device:Q_PNP_Darlington_CBE
- removed V3, V4: VSIN, symbol Simulation_SPICE:VSIN
- added Q1: PNP, symbol Simulation_SPICE:PNP
- added V1, V2: VSIN, symbol Simulation_SPICE:VSIN
- C1: value 10000u -> 4700u
- D1, D2, D3, D4: value 1N5408 -> D
- R2: value 360 -> 744
- Rload1: value 2 -> 8
Connections:
- net GND: now also V1.2, V2.2
- net In1: now also V1.1
- net In2: now also V2.1
- net Out: now also Q1.1 (C)
- net Ub: now also Q1.2 (B)
- net Vin: now also Q1.3 (E)
Other:
- note added: ".tran .1m 100m"
- note removed: ".tran .1m 200m"
