File: KiCad-Simulation-commands/KiCad-Simulation-commands.kicad_sch (KiCad schematic)
At the start: 20 parts

Commit message: Tested/updated for KiCad 9
Schematics are tested and updated for KiCad 9, no changes in circuitry
Other:
- note added: ".tran .1m 100m"
Changed lines of the file:
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@@
 (kicad_sch
-	(version 20231120)
+	(version 20250114)
 	(generator "eeschema")
-	(generator_version "8.0")
+	(generator_version "9.0")
 	(paper "A4")
 	(title_block
 		(title "KiCad Simulation commands")
-		(date "2024-12-15")
+		(date "2025-09-13")
 		(company "GitHub/OJStuff")
 	)
+	(rectangle
+		(start 13.97 127)
+		(end 175.26 160.02)
+		(stroke
+			(width 0)
+			(type default)
+		)
+		(fill
+			(type none)
+		)
+	)
+	(rectangle
+		(start 13.97 162.56)
+		(end 175.26 195.58)
+		(stroke
+			(width 0)
+			(type default)
+		)
+		(fill
+			(type none)
+		)
+	)
+	(rectangle
+		(start 13.97 55.88)
+		(end 175.26 88.9)
+		(stroke
+			(width 0)
+			(type default)
+		)
+		(fill
+			(type none)
+		)
+	)
+	(rectangle
+		(start 13.97 91.44)
+		(end 175.26 124.46)
+		(stroke
+			(width 0)
+			(type default)
+		)
+		(fill
+			(type none)
+		)
+	)
+	(rectangle
+		(start 13.97 20.32)
+		(end 175.26 53.34)
+		(stroke
+			(width 0)
+			(type default)
+		)
+		(fill
+			(type none)
+		)
+	)
+	(text ";Parameters the KiCad way"
+		(exclude_from_sim no)
+		(at 19.05 17.78 0)
+		(effects
+			(font
+				(size 1.27 1.27)
+			)
+			(justify left bottom)
+		)
+	)
+	(text ";Simulation commands"
+		(exclude_from_sim no)
+		(at 152.4 17.78 0)
+		(effects
+			(font
+				(size 1.27 1.27)
+			)
+			(justify left bottom)
+		)
+	)
+	(text ";.op"
+		(exclude_from_sim no)
+		(at 152.4 148.59 0)
+		(effects
+			(font
+				(size 1.27 1.27)
+			)
+			(justify left bottom)
+		)
+	)
+	(text ";.ac dec 1000 1 1meg"
+		(exclude_from_sim no)
+		(at 152.4 113.03 0)
+		(effects
+			(font
+				(size 1.27 1.27)
+			)
+			(justify left bottom)
+		)
+	)
+	(text ";.tran .1m 100m"
+		(exclude_from_sim no)
+		(at 152.4 78.74 0)
+		(effects
+			(font
+				(size 1.27 1.27)
+			)
+			(justify left bottom)
+		)
+	)
+	(text ".tran .1m 100m"
+		(exclude_from_sim no)
+		(at 152.4 41.91 0)
+		(effects
+			(font
+				(size 1.27 1.27)
+			)
+			(justify left bottom)
+		)
+	)
+	(text ";Parameters the PSPICE/LTSPICE way"
+		(exclude_from_sim no)
+		(at 101.854 17.526 0)
+		(effects
+			(font
+				(size 1.27 1.27)
+			)
+			(justify left bottom)
+		)
+	)
+	(text ";.dc R9 10 1k 10"
+		(exclude_from_sim no)
+		(at 152.4 181.61 0)
+		(effects
+			(font
+				(size 1.27 1.27)
+			)
+			(justify left bottom)
+		)
+	)
+	(text_box "; Examples and cheatsheet for simulation in KiCad, taken\n; from \"PSPICE Command Summary\" pdf-file.\n; \n; * * * STIMULUS TYPE * * *\n; \n; dc 0 sin(0 15 50  0  0  0)\n;  \\  \\  \\  \\  \\  \\  \\  \\  \\_ _ _  phase (phase)\n;   \\  \\  \\  \\  \\  \\  \\  \\_ _ _ _  df (damping factor)\n;    \\  \\  \\  \\  \\  \\  \\_ _ _ _ _  td (delay)\n;     \\  \\  \\  \\  \\  \\_ _ _ _ _ _  freq (frequency)\n;      \\  \\  \\  \\  \\_ _ _ _ _ _ _  va (peak amplitude voltage)\n;       \\  \\  \\  \\_ _ _ _ _ _ _ _  vo (offset voltage)\n;        \\  \\  \\_ _ _ _ _ _ _ _ _  stimulus type sinus\n;         \\  \\_ _ _ _ _ _ _ _ _ _  dc voltage (usually not needed)\n;          \\_ _ _ _ _ _ _ _ _ _ _  dc stimulus (usually not needed)\n; \n; dc 0 pulse(0  5  0  0  0  1m 2m)\n;  \\  \\    \\  \\  \\  \\  \\  \\  \\  \\_ per (periode)\n;   \\  \\    \\  \\  \\  \\  \\  \\  \\_ _ pw (pulse width)\n;    \\  \\    \\  \\  \\  \\  \\  \\_ _ _ tf (fall time)\n;     \\  \\    \\  \\  \\  \\  \\_ _ _ _ tr (rise time)\n;      \\  \\    \\  \\  \\  \\_ _ _ _ _ td (delay time)\n;       \\  \\    \\  \\  \\_ _ _ _ _ _ v2 (pulsed voltage)\n;        \\  \\    \\  \\_ _ _ _ _ _ _ v1 (initial voltage)\n;         \\  \\    \\_ _ _ _ _ _ _ _ stimulus type pulse\n;          \\  \\_ _ _ _ _ _ _ _ _ _ dc voltage (usually not needed)\n;           \\_ _ _ _ _ _ _ _ _ _ _ dc stimulus (usually not needed)\n; \n; * * * ANALYSE TYPE * * *\n; \n; .op                              dc op mode (dc compute, no plot)\n; \n; .dc V1 1 100 1\n;   \\  \\  \\  \\  \\_ _ _ _ _ _ _ _ _ variable value step\n;    \\  \\  \\  \\_ _ _ _ _ _ _ _ _ _ variable value stop\n;     \\  \\  \\_ _ _ _ _ _ _ _ _ _ _ variable value start\n;      \\  \\_ _ _ _ _ _ _ _ _ _ _ _ variable (component/source)\n;       \\_ _ _ _ _ _ _ _ _ _ _ _ _ dc analysis\n; \n; .ac lin/dec 1000 1 1meg\n;  \\      \\      \\  \\  \\_ _ _ _ _  frequency stop\n;   \\      \\      \\  \\_ _ _ _ _ _  frequency start\n;    \\      \\      \\_ _ _ _ _ _ _  points\n;     \\      \\_ _ _ _ _ _ _ _ _ _  lin or dec plot\n;      \\_ _ _ _ _ _ _ _ _ _ _ _ _  ac analysis (frequency sweep)\n; \n; .tran 1m  1\n;  \\      \\  \\_ _ _ _ _ _ _ _ _ _  end time\n;   \\      \\_ _ _ _ _ _ _ _ _ _ _  steps\n;    \\_ _ _ _ _ _ _ _ _ _ _ _ _ _  transient analysis"
+		(exclude_from_sim no)
+		(at 177.8 20.32 0)
+		(size 104.14 139.7)
+		(margins 1.125 1.125 1.125 1.125)
+		(stroke
+			(width 0)
+			(type default)
+		)
+		(fill
+			(type none)
+		)
+		(effects
+			(font
+				(face "Courier New")
+				(size 1.5 1.5)
+			)
+			(justify left top)
+		)
+	)
 	(wire
 		(pts
@@
 		)
 	)
-	(rectangle
-		(start 13.97 127)
-		(end 175.26 160.02)
-		(stroke
-			(width 0)
-			(type default)
-		)
-		(fill
-			(type none)
-		)
-	)
-	(rectangle
-		(start 13.97 162.56)
-		(end 175.26 195.58)
-		(stroke
-			(width 0)
-			(type default)
-		)
-		(fill
-			(type none)
-		)
-	)
-	(rectangle
-		(start 13.97 55.88)
-		(end 175.26 88.9)
-		(stroke
-			(width 0)
-			(type default)
-		)
-		(fill
-			(type none)
-		)
-	)
-	(rectangle
-		(start 13.97 91.44)
-		(end 175.26 124.46)
-		(stroke
-			(width 0)
-			(type default)
-		)
-		(fill
-			(type none)
-		)
-	)
-	(rectangle
-		(start 13.97 20.32)
-		(end 175.26 53.34)
-		(stroke
-			(width 0)
-			(type default)
-		)
-		(fill
-			(type none)
-		)
-	)
-	(text_box "; Examples and cheatsheet for simulation in KiCad, taken\n; from \"PSPICE Command Summary\" pdf-file.\n; \n; * * * STIMULUS TYPE * * *\n; \n; dc 0 sin(0 15 50  0  0  0)\n;  \\  \\  \\  \\  \\  \\  \\  \\  \\_ _ _  phase (phase)\n;   \\  \\  \\  \\  \\  \\  \\  \\_ _ _ _  df (damping factor)\n;    \\  \\  \\  \\  \\  \\  \\_ _ _ _ _  td (delay)\n;     \\  \\  \\  \\  \\  \\_ _ _ _ _ _  freq (frequency)\n;      \\  \\  \\  \\  \\_ _ _ _ _ _ _  va (peak amplitude voltage)\n;       \\  \\  \\  \\_ _ _ _ _ _ _ _  vo (offset voltage)\n;        \\  \\  \\_ _ _ _ _ _ _ _ _  stimulus type sinus\n;         \\  \\_ _ _ _ _ _ _ _ _ _  dc voltage (usually not needed)\n;          \\_ _ _ _ _ _ _ _ _ _ _  dc stimulus (usually not needed)\n; \n; dc 0 pulse(0  5  0  0  0  1m 2m)\n;  \\  \\    \\  \\  \\  \\  \\  \\  \\  \\_ per (periode)\n;   \\  \\    \\  \\  \\  \\  \\  \\  \\_ _ pw (pulse width)\n;    \\  \\    \\  \\  \\  \\  \\  \\_ _ _ tf (fall time)\n;     \\  \\    \\  \\  \\  \\  \\_ _ _ _ tr (rise time)\n;      \\  \\    \\  \\  \\  \\_ _ _ _ _ td (delay time)\n;       \\  \\    \\  \\  \\_ _ _ _ _ _ v2 (pulsed voltage)\n;        \\  \\    \\  \\_ _ _ _ _ _ _ v1 (initial voltage)\n;         \\  \\    \\_ _ _ _ _ _ _ _ stimulus type pulse\n;          \\  \\_ _ _ _ _ _ _ _ _ _ dc voltage (usually not needed)\n;           \\_ _ _ _ _ _ _ _ _ _ _ dc stimulus (usually not needed)\n; \n; * * * ANALYSE TYPE * * *\n; \n; .op                              dc op mode (dc compute, no plot)\n; \n; .dc V1 1 100 1\n;   \\  \\  \\  \\  \\_ _ _ _ _ _ _ _ _ variable value step\n;    \\  \\  \\  \\_ _ _ _ _ _ _ _ _ _ variable value stop\n;     \\  \\  \\_ _ _ _ _ _ _ _ _ _ _ variable value start\n;      \\  \\_ _ _ _ _ _ _ _ _ _ _ _ variable (component/source)\n;       \\_ _ _ _ _ _ _ _ _ _ _ _ _ dc analysis\n; \n; .ac lin/dec 1000 1 1meg\n;  \\      \\      \\  \\  \\_ _ _ _ _  frequency stop\n;   \\      \\      \\  \\_ _ _ _ _ _  frequency start\n;    \\      \\      \\_ _ _ _ _ _ _  points\n;     \\      \\_ _ _ _ _ _ _ _ _ _  lin or dec plot\n;      \\_ _ _ _ _ _ _ _ _ _ _ _ _  ac analysis (frequency sweep)\n; \n; .tran 1m  1\n;  \\      \\  \\_ _ _ _ _ _ _ _ _ _  end time\n;   \\      \\_ _ _ _ _ _ _ _ _ _ _  steps\n;    \\_ _ _ _ _ _ _ _ _ _ _ _ _ _  transient analysis"
-		(exclude_from_sim no)
-		(at 177.8 20.32 0)
-		(size 104.14 139.7)
-		(stroke
-			(width 0)
-			(type default)
-		)
-		(fill
-			(type none)
-		)
-		(effects
-			(font
-				(face "Courier New")
-				(size 1.5 1.5)
-			)
-			(justify left top)
-		)
-	)
-	(text ";Parameters the KiCad way"
-		(exclude_from_sim no)
-		(at 19.05 17.78 0)
-		(effects
-			(font
-				(size 1.27 1.27)
-			)
-			(justify left bottom)
-		)
-	)
-	(text ";Simulation commands"
-		(exclude_from_sim no)
-		(at 152.4 17.78 0)
-		(effects
-			(font
-				(size 1.27 1.27)
-			)
-			(justify left bottom)
-		)
-	)
-	(text ";.op"
-		(exclude_from_sim no)
-		(at 152.4 148.59 0)
-		(effects
-			(font
-				(size 1.27 1.27)
-			)
-			(justify left bottom)
-		)
-	)
-	(text ";.ac dec 1000 1 1meg"
-		(exclude_from_sim no)
-		(at 152.4 113.03 0)
-		(effects
-			(font
-				(size 1.27 1.27)
-			)
-			(justify left bottom)
-		)
-	)
-	(text ";.tran .1m 100m"
-		(exclude_from_sim no)
-		(at 152.4 78.74 0)
-		(effects
-			(font
-				(size 1.27 1.27)
-			)
-			(justify left bottom)
-		)
-	)
-	(text ";.tran .1m 100m"
-		(exclude_from_sim no)
-		(at 152.4 41.91 0)
-		(effects
-			(font
-				(size 1.27 1.27)
-			)
-			(justify left bottom)
-		)
-	)
-	(text ";Parameters the PSPICE/LTSPICE way"
-		(exclude_from_sim no)
-		(at 101.854 17.526 0)
-		(effects
-			(font
-				(size 1.27 1.27)
-			)
-			(justify left bottom)
-		)
-	)
-	(text ";.dc R9 10 1k 10"
-		(exclude_from_sim no)
-		(at 152.4 181.61 0)
-		(effects
-			(font
-				(size 1.27 1.27)
-			)
-			(justify left bottom)
-		)
-	)
 	(global_label "Out6"
 		(shape output)
@@
 		)
 	)
+	(embedded_fonts no)
 )
