File: RC-Bandpass/RC-Bandpass.kicad_sch (KiCad schematic)
At the start: 5 parts

Commit message: Tested/updated for KiCad 9
Schematics are tested and updated for KiCad 9, no changes in circuitry
Changed lines of the file:
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@@
 (kicad_sch
-	(version 20231120)
+	(version 20250114)
 	(generator "eeschema")
-	(generator_version "8.0")
+	(generator_version "9.0")
 	(paper "A4")
 	(title_block
 		(title "RC Bandpass")
-		(date "2024-12-15")
+		(date "2025-09-13")
 		(company "GitHub/OJStuff")
+	)
+	(rectangle
+		(start 121.92 76.2)
+		(end 156.21 132.08)
+		(stroke
+			(width 0)
+			(type dot)
+		)
+		(fill
+			(type none)
+		)
+	)
+	(rectangle
+		(start 162.56 76.2)
+		(end 196.85 132.08)
+		(stroke
+			(width 0)
+			(type dot)
+		)
+		(fill
+			(type none)
+		)
+	)
+	(text "Lowpass"
+		(exclude_from_sim no)
+		(at 175.26 74.93 0)
+		(effects
+			(font
+				(size 1.27 1.27)
+			)
+			(justify left bottom)
+		)
+	)
+	(text "Higpass"
+		(exclude_from_sim no)
+		(at 134.62 74.93 0)
+		(effects
+			(font
+				(size 1.27 1.27)
+			)
+			(justify left bottom)
+		)
 	)
 	(junction
@@
 			(width 0)
 			(type default)
-		)
-	)
-	(rectangle
-		(start 121.92 76.2)
-		(end 156.21 132.08)
-		(stroke
-			(width 0)
-			(type dot)
-		)
-		(fill
-			(type none)
-		)
-	)
-	(rectangle
-		(start 162.56 76.2)
-		(end 196.85 132.08)
-		(stroke
-			(width 0)
-			(type dot)
-		)
-		(fill
-			(type none)
-		)
-	)
-	(text "Lowpass"
-		(exclude_from_sim no)
-		(at 175.26 74.93 0)
-		(effects
-			(font
-				(size 1.27 1.27)
-			)
-			(justify left bottom)
-		)
-	)
-	(text "Higpass"
-		(exclude_from_sim no)
-		(at 134.62 74.93 0)
-		(effects
-			(font
-				(size 1.27 1.27)
-			)
-			(justify left bottom)
 		)
 	)
@@
 		)
 	)
+	(embedded_fonts no)
 )
