File: Rectifier-4D-Regulator-NPN/Rectifier-4D-Regulator-NPN.kicad_sch (KiCad schematic)
At the start: 14 parts, among them Q1 NPN, U1 LM317_TO-220

Commit message: Tested/updated for KiCad 9
Schematics are tested and updated for KiCad 9, no changes in circuitry
Changed lines of the file:
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@@
 (kicad_sch
-	(version 20231120)
+	(version 20250114)
 	(generator "eeschema")
-	(generator_version "8.0")
+	(generator_version "9.0")
 	(paper "A4")
 	(title_block
 		(title "Rectifier with 4 diodes, regulator and NPN passtransistor")
-		(date "2024-12-15")
+		(date "2025-09-13")
 		(company "GitHub/OJStuff")
 	)
@@
 	(label "Ub"
 		(at 184.15 71.12 0)
-		(fields_autoplaced yes)
 		(effects
 			(font
@@
 	(label "Uadj"
 		(at 161.29 88.9 0)
-		(fields_autoplaced yes)
 		(effects
 			(font
@@
 	(label "Vin"
 		(at 113.03 77.47 0)
-		(fields_autoplaced yes)
 		(effects
 			(font
@@
 		)
 	)
+	(embedded_fonts no)
 )
