File: Rectifier-4D-Zener-NPN/Rectifier-4D-Zener-NPN.kicad_sch (KiCad schematic)
At the start: 13 parts, among them Q1 NPN

Commit message: Tested/updated for KiCad 9
Schematics are tested and updated for KiCad 9, no changes in circuitry
Changed lines of the file:
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@@
 (kicad_sch
-	(version 20231120)
+	(version 20250114)
 	(generator "eeschema")
-	(generator_version "8.0")
+	(generator_version "9.0")
 	(paper "A4")
 	(title_block
 		(title "Rectifier with 4 diodes and NPN passtransistor")
-		(date "2024-12-15")
+		(date "2025-09-13")
 		(company "GitHub/OJStuff")
 	)
@@
 	(label "Vin"
 		(at 118.11 80.01 0)
-		(fields_autoplaced yes)
 		(effects
 			(font
@@
 	(label "Uz"
 		(at 161.29 99.06 0)
-		(fields_autoplaced yes)
 		(effects
 			(font
@@
 		)
 	)
+	(embedded_fonts no)
 )
