File: Rectifier-6D/Rectifier-6D.kicad_sch (KiCad schematic)
At the start: 11 parts

Commit message: Tested/updated for KiCad 9
Schematics are tested and updated for KiCad 9, no changes in circuitry
Changed lines of the file:
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@@
 (kicad_sch
-	(version 20231120)
+	(version 20250114)
 	(generator "eeschema")
-	(generator_version "8.0")
+	(generator_version "9.0")
 	(paper "A4")
 	(title_block
 		(title "Rectifier with 6 diodes (3-phase)")
-		(date "2024-12-15")
+		(date "2025-09-13")
 		(company "GitHub/OJStuff")
 	)
@@
 		)
 	)
+	(embedded_fonts no)
 )
