File: Transformer-1P-1S/Transformer-1P-1S.kicad_sch (KiCad schematic)
At the start: 5 parts

Commit message: Tested/updated for KiCad 9
Schematics are tested and updated for KiCad 9, no changes in circuitry
Changed lines of the file:
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@@
 (kicad_sch
-	(version 20231120)
+	(version 20250114)
 	(generator "eeschema")
-	(generator_version "8.0")
+	(generator_version "9.0")
 	(paper "A4")
 	(title_block
 		(title "Transformer 1P 1S")
-		(date "2024-12-15")
+		(date "2025-09-13")
 		(company "GitHub/OJStuff")
+	)
+	(rectangle
+		(start 142.24 90.17)
+		(end 146.05 110.49)
+		(stroke
+			(width 0)
+			(type default)
+		)
+		(fill
+			(type none)
+		)
+	)
+	(text "; Primary side"
+		(exclude_from_sim no)
+		(at 112.776 86.36 0)
+		(effects
+			(font
+				(size 1.27 1.27)
+			)
+			(justify left bottom)
+		)
+	)
+	(text "; Secondary side"
+		(exclude_from_sim no)
+		(at 163.83 86.36 0)
+		(effects
+			(font
+				(size 1.27 1.27)
+			)
+			(justify left bottom)
+		)
+	)
+	(text "; Up/Us = √(L1/L2)"
+		(exclude_from_sim no)
+		(at 133.858 68.326 0)
+		(effects
+			(font
+				(size 1.27 1.27)
+			)
+			(justify left bottom)
+		)
+	)
+	(text "K1 L1 L2 1.0"
+		(exclude_from_sim no)
+		(at 137.668 83.82 0)
+		(effects
+			(font
+				(size 1.27 1.27)
+			)
+			(justify left bottom)
+		)
+	)
+	(text "Transformer core"
+		(exclude_from_sim no)
+		(at 144.78 109.22 90)
+		(effects
+			(font
+				(size 1.27 1.27)
+			)
+			(justify left bottom)
+		)
+	)
+	(text "; Ideal transformer with 100% (1.0) coupling between L1 and L2"
+		(exclude_from_sim no)
+		(at 114.808 72.136 0)
+		(effects
+			(font
+				(size 1.27 1.27)
+			)
+			(justify left bottom)
+		)
 	)
 	(junction
@@
 		)
 	)
-	(rectangle
-		(start 142.24 90.17)
-		(end 146.05 110.49)
-		(stroke
-			(width 0)
-			(type default)
-		)
-		(fill
-			(type none)
-		)
-	)
-	(text "; Primary side"
-		(exclude_from_sim no)
-		(at 112.776 86.36 0)
+	(label "Vp"
+		(at 133.35 87.63 0)
 		(effects
 			(font
@@
 		)
 	)
-	(text "; Secondary side"
-		(exclude_from_sim no)
-		(at 163.83 86.36 0)
-		(effects
-			(font
-				(size 1.27 1.27)
-			)
-			(justify left bottom)
-		)
-	)
-	(text "; Up/Us = √(L1/L2)"
-		(exclude_from_sim no)
-		(at 133.858 68.326 0)
-		(effects
-			(font
-				(size 1.27 1.27)
-			)
-			(justify left bottom)
-		)
-	)
-	(text "K1 L1 L2 1.0"
-		(exclude_from_sim no)
-		(at 137.668 83.82 0)
-		(effects
-			(font
-				(size 1.27 1.27)
-			)
-			(justify left bottom)
-		)
-	)
-	(text "Transformer core"
-		(exclude_from_sim no)
-		(at 144.78 109.22 90)
-		(effects
-			(font
-				(size 1.27 1.27)
-			)
-			(justify left bottom)
-		)
-	)
-	(text "; Ideal transformer with 100% (1.0) coupling between L1 and L2"
-		(exclude_from_sim no)
-		(at 114.808 72.136 0)
-		(effects
-			(font
-				(size 1.27 1.27)
-			)
-			(justify left bottom)
-		)
-	)
-	(label "Vp"
-		(at 133.35 87.63 0)
-		(fields_autoplaced yes)
-		(effects
-			(font
-				(size 1.27 1.27)
-			)
-			(justify left bottom)
-		)
-	)
 	(label "Vs"
 		(at 154.94 87.63 0)
-		(fields_autoplaced yes)
 		(effects
 			(font
@@
 		)
 	)
+	(embedded_fonts no)
 )
