File: Transformer-1P-2S/Transformer-1P-2S.kicad_sch (KiCad schematic)
At the start: 7 parts

Commit message: Tested/updated for KiCad 9
Schematics are tested and updated for KiCad 9, no changes in circuitry
Changed lines of the file:
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@@
 (kicad_sch
-	(version 20231120)
+	(version 20250114)
 	(generator "eeschema")
-	(generator_version "8.0")
+	(generator_version "9.0")
 	(paper "A4")
 	(title_block
 		(title "Transformer 1P 2S")
-		(date "2024-12-15")
+		(date "2025-09-13")
 		(company "GitHub/OJStuff")
+	)
+	(rectangle
+		(start 144.78 90.17)
+		(end 148.59 110.49)
+		(stroke
+			(width 0)
+			(type default)
+		)
+		(fill
+			(type none)
+		)
+	)
+	(text "; Up/Us1 = √(L1/L2)\n; Up/Us2 = √(L1/L3)"
+		(exclude_from_sim no)
+		(at 135.636 64.516 0)
+		(effects
+			(font
+				(size 1.27 1.27)
+			)
+			(justify left bottom)
+		)
+	)
+	(text "; Secondary side"
+		(exclude_from_sim no)
+		(at 166.37 86.36 0)
+		(effects
+			(font
+				(size 1.27 1.27)
+			)
+			(justify left bottom)
+		)
+	)
+	(text "K1 L1 L2 1.0\nK2 L1 L3 1.0\nK3 L2 L3 1.0"
+		(exclude_from_sim no)
+		(at 139.7 82.804 0)
+		(effects
+			(font
+				(size 1.27 1.27)
+			)
+			(justify left bottom)
+		)
+	)
+	(text "Transformer core"
+		(exclude_from_sim no)
+		(at 147.32 109.22 90)
+		(effects
+			(font
+				(size 1.27 1.27)
+			)
+			(justify left bottom)
+		)
+	)
+	(text "; Primary side"
+		(exclude_from_sim no)
+		(at 115.316 86.36 0)
+		(effects
+			(font
+				(size 1.27 1.27)
+			)
+			(justify left bottom)
+		)
+	)
+	(text "; Ideal transformer with 100% (1.0) coupling between L1, L2 and 3"
+		(exclude_from_sim no)
+		(at 114.046 70.866 0)
+		(effects
+			(font
+				(size 1.27 1.27)
+			)
+			(justify left bottom)
+		)
 	)
 	(junction
@@
 		)
 	)
-	(rectangle
-		(start 144.78 90.17)
-		(end 148.59 110.49)
-		(stroke
-			(width 0)
-			(type default)
-		)
-		(fill
-			(type none)
-		)
-	)
-	(text "; Up/Us1 = √(L1/L2)\n; Up/Us2 = √(L1/L3)"
-		(exclude_from_sim no)
-		(at 135.636 64.516 0)
-		(effects
-			(font
-				(size 1.27 1.27)
-			)
-			(justify left bottom)
-		)
-	)
-	(text "; Secondary side"
-		(exclude_from_sim no)
-		(at 166.37 86.36 0)
-		(effects
-			(font
-				(size 1.27 1.27)
-			)
-			(justify left bottom)
-		)
-	)
-	(text "K1 L1 L2 1.0\nK2 L1 L3 1.0\nK3 L2 L3 1.0"
-		(exclude_from_sim no)
-		(at 139.7 82.804 0)
-		(effects
-			(font
-				(size 1.27 1.27)
-			)
-			(justify left bottom)
-		)
-	)
-	(text "Transformer core"
-		(exclude_from_sim no)
-		(at 147.32 109.22 90)
-		(effects
-			(font
-				(size 1.27 1.27)
-			)
-			(justify left bottom)
-		)
-	)
-	(text "; Primary side"
-		(exclude_from_sim no)
-		(at 115.316 86.36 0)
-		(effects
-			(font
-				(size 1.27 1.27)
-			)
-			(justify left bottom)
-		)
-	)
-	(text "; Ideal transformer with 100% (1.0) coupling between L1, L2 and 3"
-		(exclude_from_sim no)
-		(at 114.046 70.866 0)
-		(effects
-			(font
-				(size 1.27 1.27)
-			)
-			(justify left bottom)
-		)
-	)
 	(label "Vp"
 		(at 135.89 87.63 0)
-		(fields_autoplaced yes)
-		(effects
-			(font
-				(size 1.27 1.27)
-			)
-			(justify left bottom)
-		)
-	)
-	(label "Vs2"
-		(at 157.48 113.03 0)
-		(fields_autoplaced yes)
-		(effects
-			(font
-				(size 1.27 1.27)
-			)
-			(justify left bottom)
-		)
-	)
-	(label "Vs1"
-		(at 157.48 87.63 0)
-		(fields_autoplaced yes)
 		(effects
 			(font
@@
 		)
 	)
+	(embedded_fonts no)
 )
